File: minimal_adp1031/minimal_adp1031.kicad_sch (KiCad schematic)
At the start: 0 parts

Commit message: backup
Parts:
- added C1: 4.7 µF, capacitor_footprints:C_1210_200_3225Metric, symbol UNITED_CAPACITORS_DATA_BASE:C_GCM32DC72A475KE02K
- added C2, C3, C4: 100 nF, capacitor_footprints:C_0402_1005Metric, symbol UNITED_CAPACITORS_DATA_BASE:C_GCM155R71H104KE02D
- added C5: 4.7 µF, capacitor_footprints:C_0603_1608Metric, symbol UNITED_CAPACITORS_DATA_BASE:C_C1608X7S1A475K080AC
- added C6, C7, C8: 10 µF, capacitor_footprints:C_1206_3216Metric, symbol UNITED_CAPACITORS_DATA_BASE:C_CL31B106KBHNNN#
- added D1: 62.0 V, diode_footprints:SOD_123, symbol UNITED_DIODES_DATA_BASE:D_MMSZ5265BT1G
- added D2: 100.0 V, diode_footprints:PowerDI_123, symbol UNITED_DIODES_DATA_BASE:D_DFLS1200-7
- added D3: 200.0 V, diode_footprints:SOD_123F, symbol UNITED_DIODES_DATA_BASE:D_US1DWF
- added FID1, FID2, FID3: Fiducial, no_components_footprints:Fiducial_0.5mm_Mask1mm, symbol UNITED_NO_COMPONENTS_DATA_BASE:Fiducial
- added JP1: SolderJumper_3_Open, solder_jumper_footprints:SolderJumper-3_P1.3mm_Open_RoundedPad1.0x1.5mm_NumberLabels, symbol UNITED_SOLDER_JUMPERS:SolderJumper_3_Open
- added JP2, JP3, JP4: SolderJumper_2_Bridged, solder_jumper_footprints:SolderJumper-2_P1.3mm_Bridged_RoundedPad1.0x1.5mm, symbol UNITED_SOLDER_JUMPERS:SolderJumper_2_Bridged
- added L1, L2: 100 µH, inductor_footprints:XFL3012, symbol UNITED_INDUCTORS_DATA_BASE:L_XFL3012-104ME
- added R1, R2, R3, R4, R5, R6, R7, R8: 100 kΩ, resistor_footprints:R_0402_1005Metric, symbol UNITED_RESISTORS_DATA_BASE:R_ERJ-2GEJ104X
- added R10: 120 kΩ, resistor_footprints:R_0402_1005Metric, symbol UNITED_RESISTORS_DATA_BASE:R_ERJ-2RKF1203X
- added R11: 2.15 MΩ, resistor_footprints:R_0402_1005Metric, symbol UNITED_RESISTORS_DATA_BASE:R_RC0402FR-072M15L
- added R12: 121 kΩ, resistor_footprints:R_0402_1005Metric, symbol UNITED_RESISTORS_DATA_BASE:R_ERJ-2RKF1213X
- added R9: 3.48 MΩ, resistor_footprints:R_0402_1005Metric, symbol UNITED_RESISTORS_DATA_BASE:R_RC0402FR-073M48L
- added T1: ZA9644-AED, transformer_footprints:ZA9644, symbol UNITED_TRANSFORMERS_DATA_BASE:T_ZA9644-AED
- added U1: ADP1031ACPZ-3-R7, analog_devices_footprints:CP-41-1_ADI, symbol UNITED_IC_ADI:U_ADP1031ACPZ-3-R7
Connections:
- new net: D1.1, D2.1
- new net: D3.2, T1.5
- new net -15V0: JP4.2
- new net 3V3: C3.1, C4.1, JP2.2, R4.1, R5.1, R7.1, U1.10 (SVDD1), U1.20 (SVDD2), U1.26 (DNC)
- new net FB1: R10.1, R9.2, U1.19 (FB1)
- new net FB3: R11.1, R12.2, U1.11 (FB3)
- new net GND: C1.1, JP1.3 (B), U1.28 (PGNDP), U1.33 (GNDP), U1.43 (EPGNDP)
- new net GNDA: C3.2, C4.2, C5.2, C6.2, C7.2, C8.2, L2.2, R10.2, R11.2, R2.2, R3.2, R6.2, R8.1, T1.8, U1.16 (SGND2), U1.27 (SGND2), U1.4 (SGND2), U1.44 (EPGND2), U1.5 (SGND1)
- new net GNDD: C2.2, U1.3 (MGND), U1.34 (MGND), U1.42 (EPGNDM)
- new net MCK: U1.40 (MCK)
- new net MGPI1: U1.36 (MGPI1)
- new net MGPI2: U1.37 (MGPI2)
- new net MGPO3: U1.38 (MGPO3)
- new net MI: U1.1 (MI)
- new net MO: U1.41 (MO)
- new net MVDD: C2.1, R1.1, U1.39 (MVDD)
- new net PWRGD: R1.2, U1.35 (PWRGD)
- new net SCK: R4.2, U1.9 (SCK)
- new net SGPI3: R5.2, U1.21 (SGPI3)
- new net SGPO1: R7.2, U1.23 (SGPO1)
- new net SGPO2: R6.1, U1.22 (SGPO2)
- new net SI: R3.1, U1.8 (SI)
- new net SLEW: JP1.2 (C), U1.32 (SLEW)
- new net SO: R2.1, U1.7 (SO)
- new net SW2: L1.1, U1.17 (SW2)
- new net SW3: L2.1, U1.13 (SW3)
- new net SWP: D2.2, T1.4, U1.29 (SWP)
- new net SYNC: R8.2, U1.14 (SYNC)
- new net VDD_24V: JP3.2
- new net VINP: C1.2, D1.2, JP1.1 (A), T1.1, U1.30 (VINP), U1.31 (EN)
- new net VOUT1: C6.1, C7.1, D3.1, JP3.1, R9.1, U1.18 (VOUT1)
- new net VOUT2: C5.1, JP2.1, L1.2, U1.15 (VOUT2)
- new net VOUT3: C8.1, JP4.1, R12.1, U1.12 (VOUT3)
- new net ~{MSS}: U1.2 (~{MSS})
- new net ~{SSS}: U1.6 (~{SSS})

Commit message: backup
Parts:
- added J1, J2, J4, J5, J6: FW-02-03-G-D-085-155, connector_footprints:FW-02-03-G-D-085-155, symbol UNITED_CONNECTORS_DATA_BASE:J_FW-02-03-G-D-085-155
- added J3, J7: FW-08-03-G-D-085-155, connector_footprints:FW-08-03-G-D-085-155, symbol UNITED_CONNECTORS_DATA_BASE:J_FW-08-03-G-D-085-155
- added TP1, TP10, TP11, TP12, TP13, TP14, TP15, TP16, TP17, TP18, TP19, TP2, TP20, TP21, TP22, TP23, TP24, TP25, TP26, TP3, TP4, TP5, TP6, TP7, TP8, TP9: TestPoint, test_point_footprints:TestPoint_THTPad_Castelated, symbol UNITED_TEST_POINTS:TestPoint_Castelated
Connections:
- net -15V0: now also J4.2, J4.4, TP25.1
- net 3V3: now also J5.1, J5.3, TP22.1
- net GND: now also J2.2, J2.4, TP3.1
- net GNDA: now also J4.1, J4.3, J5.2, J5.4, J6.2, J6.4, J7.1, J7.10, J7.12, J7.14, J7.16, J7.2, J7.4, J7.6, J7.8, TP13.1, TP21.1, TP24.1, TP26.1
- net GNDD: now also J1.2, J1.4, J3.1, J3.11, J3.13, J3.15, J3.2, J3.3, J3.5, J3.7, J3.9, TP1.1, TP5.1
- net MCK: now also J3.10, TP9.1
- net MGPI1: now also J3.16, TP12.1
- net MGPI2: now also J3.14, TP11.1
- net MGPO3: now also J3.12, TP10.1
- net MI: now also J3.6, TP7.1
- net MO: now also J3.8, TP8.1
- net MVDD: now also J1.1, J1.3, TP2.1
- net SCK: now also J7.9, TP17.1
- net SGPI3: now also J7.11, TP18.1
- net SGPO1: now also J7.15, TP20.1
- net SGPO2: now also J7.13, TP19.1
- net SI: now also J7.7, TP16.1
- net SO: now also J7.5, TP15.1
- net VDD_24V: now also J6.1, J6.3, TP23.1
- net VINP: now also J2.1, J2.3, TP4.1
- net ~{MSS}: now also J3.4, TP6.1
- net ~{SSS}: now also J7.3, TP14.1
Other:
- moved on the sheet: C1, C2, C3, C4, C5, C6, C7, C8, D1, D2, D3, FID1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

Commit message: backup
Parts:
- added MB1, MB2, MB3, MB4, MB5: mouse-bite-midle-50mil-200mil, mouse_bite_footprints:mouse-bite-50mil-305mil, symbol UNITED_MOUSE_BITES_DATA_BASE:mouse-bite-50mil-305mil
- added MB6, MB7: mouse-bite-50mil-450mil, mouse_bite_footprints:mouse-bite-50mil-500mil, symbol UNITED_MOUSE_BITES_DATA_BASE:mouse-bite-50mil-500mil
- U1: value ADP1031ACPZ-3-R7 -> ADP1031ACPZ-2-R7; symbol UNITED_IC_ADI:U_ADP1031ACPZ-3-R7 -> UNITED_IC_ADI:U_ADP1031ACPZ-2-R7; MPN ADP1031ACPZ-3-R7 -> ADP1031ACPZ-2-R7
Connections:
- net 3V3 renamed 5V0

Commit message: backup
Parts:
- renumbered C6 to C3, C3 to C4, C4 to C5, C5 to C6, FID3 to FID1, FID1 to FID2, FID2 to FID3, J7 to J4, J4 to J5, J5 to J6, J6 to J7, JP4 to JP2, JP2 to JP3, JP3 to JP4, L2 to L1, L1 to L2, MB5 to MB1, MB4 to MB2, MB7 to MB3, MB6 to MB4, MB3 to MB5, MB1 to MB6, MB2 to MB7, R11 to R10, R12 to R11, R10 to R12, TP26 to TP21, TP25 to TP22, TP22 to TP23, TP21 to TP24, TP23 to TP25, TP24 to TP26
Changed lines of the file:
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@@
 		(dnp no)
 		(fields_autoplaced yes)
-		(property "Reference" "TP22"
+		(property "Reference" "TP23"
 			(at 294.64 93.2179 0)
 			(effects
@@
 			(project "minimal_adp1031"
 				(path "/9c9a963e-fcf2-442a-88cc-38bcf1c7456f"
-					(reference "TP22")
+					(reference "TP23")
 					(unit 1)
 				)
@@
 		(dnp no)
 		(fields_autoplaced yes)
-		(property "Reference" "MB2"
+		(property "Reference" "MB7"
 			(at 360.68 66.04 0)
 			(effects
@@
 			(project "minimal_adp1031"
 				(path "/9c9a963e-fcf2-442a-88cc-38bcf1c7456f"
-					(reference "MB2")
+					(reference "MB7")
 					(unit 1)
 				)
@@
 		(dnp no)
 		(fields_autoplaced yes)
-		(property "Reference" "TP26"
+		(property "Reference" "TP21"
 			(at 307.34 131.3179 0)
 			(effects
@@
 			(project "minimal_adp1031"
 				(path "/9c9a963e-fcf2-442a-88cc-38bcf1c7456f"
-					(reference "TP26")
+					(reference "TP21")
 					(unit 1)
 				)
@@
 		(dnp no)
 		(fields_autoplaced yes)
-		(property "Reference" "FID2"
+		(property "Reference" "FID3"
 			(at 104.14 194.3099 0)
 			(effects
@@
 			(project "minimal_adp1031"
 				(path "/9c9a963e-fcf2-442a-88cc-38bcf1c7456f"
-					(reference "FID2")
+					(reference "FID3")
 					(unit 1)
 				)
@@
 		(dnp no)
 		(fields_autoplaced yes)
-		(property "Reference" "FID1"
+		(property "Reference" "FID2"
 			(at 91.44 194.3099 0)
 			(effects
@@
 			(project "minimal_adp1031"
 				(path "/9c9a963e-fcf2-442a-88cc-38bcf1c7456f"
-					(reference "FID1")
+					(reference "FID2")
 					(unit 1)
 				)
@@
 		(dnp no)
 		(fields_autoplaced yes)
-		(property "Reference" "C3"
+		(property "Reference" "C4"
 			(at 241.3 175.26 0)
 			(effects
@@
 			(project "minimal_adp1031"
 				(path "/9c9a963e-fcf2-442a-88cc-38bcf1c7456f"
-					(reference "C3")
+					(reference "C4")
 					(unit 1)
 				)
@@
 		(dnp no)
 		(fields_autoplaced yes)
-		(property "Reference" "JP4"
+		(property "Reference" "JP2"
 			(at 285.75 120.65 0)
 			(effects
@@
 			(project "minimal_adp1031"
 				(path "/9c9a963e-fcf2-442a-88cc-38bcf1c7456f"
-					(reference "JP4")
+					(reference "JP2")
 					(unit 1)
 				)
@@
 		(dnp no)
 		(fields_autoplaced yes)
-		(property "Reference" "J4"
+		(property "Reference" "J5"
 			(at 335.28 129.5399 90)
 			(effects
@@
 			(project "minimal_adp1031"
 				(path "/9c9a963e-fcf2-442a-88cc-38bcf1c7456f"
-					(reference "J4")
+					(reference "J5")
 					(unit 1)
 				)
@@
 		(dnp no)
 		(fields_autoplaced yes)
-		(property "Reference" "TP23"
+		(property "Reference" "TP25"
 			(at 307.34 52.5779 0)
 			(effects
@@
 			(project "minimal_adp1031"
 				(path "/9c9a963e-fcf2-442a-88cc-38bcf1c7456f"
-					(reference "TP23")
+					(reference "TP25")
 					(unit 1)
 				)
@@
 		(dnp no)
 		(fields_autoplaced yes)
-		(property "Reference" "TP21"
+		(property "Reference" "TP24"
 			(at 294.64 105.9179 0)
 			(effects
@@
 			(project "minimal_adp1031"
 				(path "/9c9a963e-fcf2-442a-88cc-38bcf1c7456f"
-					(reference "TP21")
+					(reference "TP24")
 					(unit 1)
 				)
@@
 		(dnp no)
 		(fields_autoplaced yes)
-		(property "Reference" "JP3"
+		(property "Reference" "JP4"
 			(at 292.1 54.61 0)
 			(effects
@@
 			(project "minimal_adp1031"
 				(path "/9c9a963e-fcf2-442a-88cc-38bcf1c7456f"
-					(reference "JP3")
+					(reference "JP4")
 					(unit 1)
 				)
@@
 		(dnp no)
 		(fields_autoplaced yes)
-		(property "Reference" "MB3"
+		(property "Reference" "MB5"
 			(at 359.41 152.4 0)
 			(effects
@@
 			(project "minimal_adp1031"
 				(path "/9c9a963e-fcf2-442a-88cc-38bcf1c7456f"
-					(reference "MB3")
+					(reference "MB5")
 					(unit 1)
 				)
@@
 		(on_board yes)
 		(dnp no)
-		(property "Reference" "R11"
+		(property "Reference" "R10"
 			(at 256.54 144.7801 90)
 			(effects
@@
 			(project ""
 				(path "/9c9a963e-fcf2-442a-88cc-38bcf1c7456f"
-					(reference "R11")
+					(reference "R10")
 					(unit 1)
 				)
@@
 		(on_board yes)
 		(dnp no)
-		(property "Reference" "J6"
+		(property "Reference" "J7"
 			(at 335.28 66.0401 90)
 			(effects
@@
 			(project "minimal_adp1031"
 				(path "/9c9a963e-fcf2-442a-88cc-38bcf1c7456f"
-					(reference "J6")
+					(reference "J7")
 					(unit 1)
 				)
@@
 		(dnp no)
 		(fields_autoplaced yes)
-		(property "Reference" "J7"
+		(property "Reference" "J4"
 			(at 266.7 191.77 0)
 			(effects
@@
 			(project "minimal_adp1031"
 				(path "/9c9a963e-fcf2-442a-88cc-38bcf1c7456f"
-					(reference "J7")
+					(reference "J4")
 					(unit 1)
 				)
@@
 		(dnp no)
 		(fields_autoplaced yes)
-		(property "Reference" "L2"
+		(property "Reference" "L1"
 			(at 243.84 143.51 0)
 			(effects
@@
 			(project "minimal_adp1031"
 				(path "/9c9a963e-fcf2-442a-88cc-38bcf1c7456f"
-					(reference "L2")
+					(reference "L1")
 					(unit 1)
 				)
@@
 		(dnp no)
 		(fields_autoplaced yes)
-		(property "Reference" "TP25"
+		(property "Reference" "TP22"
 			(at 307.34 118.6179 0)
 			(effects
@@
 			(project "minimal_adp1031"
 				(path "/9c9a963e-fcf2-442a-88cc-38bcf1c7456f"
-					(reference "TP25")
+					(reference "TP22")
 					(unit 1)
 				)
@@
 		(dnp no)
 		(fields_autoplaced yes)
-		(property "Reference" "C4"
+		(property "Reference" "C5"
 			(at 247.65 165.1 0)
 			(effects
@@
 			(project "minimal_adp1031"
 				(path "/9c9a963e-fcf2-442a-88cc-38bcf1c7456f"
-					(reference "C4")
+					(reference "C5")
 					(unit 1)
 				)
@@
 		(dnp no)
 		(fields_autoplaced yes)
-		(property "Reference" "MB4"
+		(property "Reference" "MB2"
 			(at 91.44 69.85 0)
 			(effects
@@
 			(project "minimal_adp1031"
 				(path "/9c9a963e-fcf2-442a-88cc-38bcf1c7456f"
-					(reference "MB4")
+					(reference "MB2")
 					(unit 1)
 				)
@@
 		(dnp no)
 		(fields_autoplaced yes)
-		(property "Reference" "MB5"
+		(property "Reference" "MB1"
 			(at 105.41 168.91 0)
 			(effects
@@
 			(project "minimal_adp1031"
 				(path "/9c9a963e-fcf2-442a-88cc-38bcf1c7456f"
-					(reference "MB5")
+					(reference "MB1")
 					(unit 1)
 				)
@@
 		(on_board yes)
 		(dnp no)
-		(property "Reference" "R10"
+		(property "Reference" "R12"
 			(at 233.68 62.23 0)
 			(effects
@@
 			(project ""
 				(path "/9c9a963e-fcf2-442a-88cc-38bcf1c7456f"
-					(reference "R10")
+					(reference "R12")
 					(unit 1)
 				)
@@
 		(dnp no)
 		(fields_autoplaced yes)
-		(property "Reference" "JP2"
+		(property "Reference" "JP3"
 			(at 273.05 95.25 0)
 			(effects
@@
 			(project "minimal_adp1031"
 				(path "/9c9a963e-fcf2-442a-88cc-38bcf1c7456f"
-					(reference "JP2")
+					(reference "JP3")
 					(unit 1)
 				)
@@
 		(dnp no)
 		(fields_autoplaced yes)
-		(property "Reference" "MB1"
+		(property "Reference" "MB6"
 			(at 351.79 105.41 0)
 			(effects
@@
 			(project ""
 				(path "/9c9a963e-fcf2-442a-88cc-38bcf1c7456f"
-					(reference "MB1")
+					(reference "MB6")
 					(unit 1)
 				)
@@
 		(dnp no)
 		(fields_autoplaced yes)
-		(property "Reference" "L1"
+		(property "Reference" "L2"
 			(at 243.84 106.68 0)
 			(effects
@@
 			(project "minimal_adp1031"
 				(path "/9c9a963e-fcf2-442a-88cc-38bcf1c7456f"
-					(reference "L1")
+					(reference "L2")
 					(unit 1)
 				)
@@
 		(dnp no)
 		(fields_autoplaced yes)
-		(property "Reference" "FID3"
+		(property "Reference" "FID1"
 			(at 116.84 194.3099 0)
 			(effects
@@
 			(project "minimal_adp1031"
 				(path "/9c9a963e-fcf2-442a-88cc-38bcf1c7456f"
-					(reference "FID3")
+					(reference "FID1")
 					(unit 1)
 				)
@@
 		(dnp no)
 		(fields_autoplaced yes)
-		(property "Reference" "C6"
+		(property "Reference" "C3"
 			(at 283.21 62.2299 90)
 			(effects
@@
 			(project "minimal_adp1031"
 				(path "/9c9a963e-fcf2-442a-88cc-38bcf1c7456f"
-					(reference "C6")
+					(reference "C3")
 					(unit 1)
 				)
@@
 		(dnp no)
 		(fields_autoplaced yes)
-		(property "Reference" "MB6"
+		(property "Reference" "MB4"
 			(at 266.7 226.06 0)
 			(effects
@@
 			(project "minimal_adp1031"
 				(path "/9c9a963e-fcf2-442a-88cc-38bcf1c7456f"
-					(reference "MB6")
+					(reference "MB4")
 					(unit 1)
 				)
@@
 		(dnp no)
 		(fields_autoplaced yes)
-		(property "Reference" "C5"
+		(property "Reference" "C6"
 			(at 257.81 109.2199 90)
 			(effects
@@
 			(project "minimal_adp1031"
 				(path "/9c9a963e-fcf2-442a-88cc-38bcf1c7456f"
-					(reference "C5")
+					(reference "C6")
 					(unit 1)
 				)
@@
 		(dnp no)
 		(fields_autoplaced yes)
-		(property "Reference" "J5"
+		(property "Reference" "J6"
 			(at 309.88 104.1399 90)
 			(effects
@@
 			(project "minimal_adp1031"
 				(path "/9c9a963e-fcf2-442a-88cc-38bcf1c7456f"
-					(reference "J5")
+					(reference "J6")
 					(unit 1)
 				)
@@
 		(dnp no)
 		(fields_autoplaced yes)
-		(property "Reference" "MB7"
+		(property "Reference" "MB3"
 			(at 165.1 226.06 0)
 			(effects
@@
 			(project "minimal_adp1031"
 				(path "/9c9a963e-fcf2-442a-88cc-38bcf1c7456f"
-					(reference "MB7")
+					(reference "MB3")
 					(unit 1)
 				)
@@
 		(on_board yes)
 		(dnp no)
-		(property "Reference" "R12"
+		(property "Reference" "R11"
 			(at 256.54 132.0801 90)
 			(effects
@@
 			(project ""
 				(path "/9c9a963e-fcf2-442a-88cc-38bcf1c7456f"
-					(reference "R12")
+					(reference "R11")
 					(unit 1)
 				)
@@
 		(dnp no)
 		(fields_autoplaced yes)
-		(property "Reference" "TP24"
+		(property "Reference" "TP26"
 			(at 307.34 65.2779 0)
 			(effects
@@
 			(project "minimal_adp1031"
 				(path "/9c9a963e-fcf2-442a-88cc-38bcf1c7456f"
-					(reference "TP24")
+					(reference "TP26")
 					(unit 1)
 				)
